Commit message: fix error

File: Project2/src/my_robot/urdf/my_robot.xacro (robot description, xacro)
@@ -16,5 +16,5 @@
     <pose>0 0 0 0 0 0</pose>
     <inertial>
-      <mass value="1.5"/>
+      <mass value="5"/>
       <origin xyz="0.0 0 0" rpy=" 0 0 0"/>
       <inertia
@@ -59,5 +59,5 @@
        <origin xyz="0 0 0" rpy=" 1.5707 0 0"/>
         <geometry>
-          <cylinder radius="0.1" length="0.01" />
+          <cylinder radius="0.1" length="0.1" />
         </geometry>
     </visual>
@@ -65,5 +65,5 @@
        <origin xyz="0 0 0" rpy=" 1.5707 0 0"/>
         <geometry>
-          <cylinder radius="0.1" length="0.01" />
+          <cylinder radius="0.1" length="0.1" />
         </geometry>
     </collision>
@@ -91,5 +91,5 @@
        <origin xyz="0 0 0" rpy=" 1.5707 0 0"/>
         <geometry>
-          <cylinder radius="0.1"       length="0.01" />
+          <cylinder radius="0.1" length="0.1" />
         </geometry>
       </visual>
@@ -97,5 +97,5 @@
        <origin xyz="0 0 0" rpy=" 1.5707 0 0"/>
         <geometry>
-          <cylinder radius="0.1"       length="0.01" />
+          <cylinder radius="0.1" length="0.1" />
         </geometry>
     </collision>
@@ -123,5 +123,5 @@
        <origin xyz="0 0 0" rpy=" 1.5707 0 0"/>
         <geometry>
-          <cylinder radius="0.1"       length="0.01" />
+          <cylinder radius="0.1" length="0.1" />
         </geometry>
       </visual>
@@ -129,5 +129,5 @@
        <origin xyz="0 0 0" rpy=" 1.5707 0 0"/>
         <geometry>
-          <cylinder radius="0.1"       length="0.01" />
+          <cylinder radius="0.1" length="0.1" />
         </geometry>
     </collision>
@@ -155,5 +155,5 @@
        <origin xyz="0 0 0" rpy=" 1.5707 0 0"/>
         <geometry>
-          <cylinder radius="0.1"       length="0.01" />
+          <cylinder radius="0.1" length="0.1" />
         </geometry>
       </visual>
@@ -161,5 +161,5 @@
        <origin xyz="0 0 0" rpy=" 1.5707 0 0"/>
         <geometry>
-          <cylinder radius="0.1"       length="0.01" />
+          <cylinder radius="0.1" length="0.1" />
         </geometry>
     </collision>
